File: pe/kicad-template/template.kicad_sch (KiCad schematic)
At the start: 21 parts, among them U1 TPS542025DDCR

Commit message: Revert "PE Onboarding Project - Christian Walter"
This reverts commit c39510325f63961227da3eea3b54a31334393b75.
Parts:
- removed C1, C11, C12, C13, C14, C15, C16, C17: 22 µF, 0603B103K500CT:CAPC1608X87N, symbol 0603B103K500CT:0603B103K500CT
- removed C10, C18, C19: 0.1 µF, C0603C104K5RACTU:CAPC1608X90, symbol C0603C104K5RACTU:C0603C104K5RACTU
- removed C2, C3, C4, C5, C6, C7, C8, C9: 10 µF, TMK107BBJ106MA-T:CAPC1709X100N, symbol TMK107BBJ106MA-T:TMK107BBJ106MA-T
- removed L1: 15 µH, 0640CDMCCDS-150MC Mimic:IND_ETQ-P5M470YFK, symbol ETQ-P5M470YFK:ETQ-P5M470YFK
- removed U1: TPS542025DDCR, Package_TO_SOT_SMD:SOT-23-6, symbol Regulator_Switching:TPS54202DDC

Commit message: PE Onboarding Project - Christian Walter
Parts:
- added C1, C11, C12, C13, C14, C15, C16, C17: 22 µF, 0603B103K500CT:CAPC1608X87N, symbol 0603B103K500CT:0603B103K500CT
- added C10, C18, C19: 0.1 µF, C0603C104K5RACTU:CAPC1608X90, symbol C0603C104K5RACTU:C0603C104K5RACTU
- added C2, C3, C4, C5, C6, C7, C8, C9: 10 µF, TMK107BBJ106MA-T:CAPC1709X100N, symbol TMK107BBJ106MA-T:TMK107BBJ106MA-T
- added L1: 15 µH, 0640CDMCCDS-150MC Mimic:IND_ETQ-P5M470YFK, symbol ETQ-P5M470YFK:ETQ-P5M470YFK
- added U1: TPS542025DDCR, Package_TO_SOT_SMD:SOT-23-6, symbol Regulator_Switching:TPS54202DDC
Connections:
- new net: C19.1, U1.6 (BOOT)
- new net: C19.2, L1.1, U1.2 (SW)
- new net +12V: C10.1, C2.1, C3.1, C4.1, C5.1, C6.1, C7.1, C8.1, C9.1, U1.3 (VIN)
- new net +5V: C1.2, C11.2, C12.2, C13.2, C14.2, C15.2, C16.2, C17.2, C18.2, L1.2, U1.4 (FB)
- new net GND: C1.1, C10.2, C11.1, C12.1, C13.1, C14.1, C15.1, C16.1, C17.1, C18.1, C2.2, C3.2, C4.2, C5.2, C6.2, C7.2, C8.2, C9.2, U1.1 (GND)
